Commit message: modified urdf servos zero points

File: models/dofbot_urdf_with_gripper/dofbot_with_gripper.urdf (robot description, URDF)
Before this commit: robot dofbot_model_4, 12 links, 11 joints
Joints:
- joint joint1: limit lower=-1.57 upper=1.57 effort=0 velocity=0 -> lower=-3.14 upper=3.14 effort=0 velocity=0; origin xyz=0.073174 0 0.082 rpy=0 0 0 -> xyz=0.073174 0 0.082 rpy=0 0 1.57
- joint joint2: limit lower=-1.57 upper=1.57 effort=0 velocity=0 -> lower=0.0 upper=3.14 effort=0 velocity=0; origin xyz=0 -0.0183 0.0255 rpy=0 0 0 -> xyz=0 -0.0183 0.0255 rpy=0 -1.57 0
- joint joint3: limit lower=-2.62 upper=2.62 effort=0 velocity=0 -> lower=-1.05 upper=4.19 effort=0 velocity=0; origin xyz=0 0 0.08285 rpy=0 0 0 -> xyz=0 0 0.08285 rpy=0 -1.57 0
- joint joint4: limit lower=-1.73 upper=1.73 effort=0 velocity=0 -> lower=-0.16 upper=3.3 effort=0 velocity=0; origin xyz=0 0.000599999999990254 0.0828499999999967 rpy=0 0 0 -> xyz=0 0.000599999999990254 0.0828499999999967 rpy=0 -1.57 0
- joint joint5: origin xyz=-0.00216911459875002 0.0183050000000032 0.0816240000000007 rpy=0 0 0 -> xyz=-0.00216911459875002 0.0183050000000032 0.0816240000000007 rpy=0 0 -1.57
